File: pcb/hdmi-breakout/hdmi-breakout.kicad_pcb (KiCad board)
At the start: 4 copper layers, 35 x 29 mm, 4 parts, among them J2 HDMI_A_1.4, J3 HDMI_A_1.4

Commit message: update docs
Parts:
- J1, J4: value ~ -> Conn_01x09
